File: hardware/winch-link/winch-link.kicad_sch (KiCad schematic)
At the start: 41 parts, among them J1 USB_C_Receptacle_USB2.0, J2 Conn_01x02_Pin, J3 Conn_01x02_Pin, J4 VBAT, J5 display conn, J6 BAT GND, Q1 AO3401A, SW1 RST, SW2 PRG, U1 RFM95W-868S2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

Commit message: Add BOM and CPL files
Parts:
- J2, J3, J4, J5, J6, PCB_Antenna1: now left out of the parts list
Changed lines of the file:
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@@
   )
   (symbol (lib_id "Connector:Conn_01x02_Pin") (at 160.02 55.88 0) (unit 1)
-    (in_bom yes) (on_board yes) (dnp no) (fields_autoplaced)
+    (in_bom no) (on_board yes) (dnp no) (fields_autoplaced)
     (property "Reference" "J2" (at 160.655 52.07 0)
       (effects (font (size 1.27 1.27)))
@@
   )
   (symbol (lib_id "Connector:Conn_01x01_Pin") (at 328.295 236.855 0) (unit 1)
-    (in_bom yes) (on_board yes) (dnp no) (fields_autoplaced)
+    (in_bom no) (on_board yes) (dnp no) (fields_autoplaced)
     (property "Reference" "J4" (at 328.93 233.045 0)
       (effects (font (size 1.27 1.27)))
@@
   )
   (symbol (lib_id "Connector:Conn_01x02_Pin") (at 214.63 57.15 0) (unit 1)
-    (in_bom yes) (on_board yes) (dnp no) (fields_autoplaced)
+    (in_bom no) (on_board yes) (dnp no) (fields_autoplaced)
     (property "Reference" "J3" (at 215.265 53.34 0)
       (effects (font (size 1.27 1.27)))
@@
   )
   (symbol (lib_id "Connector:Conn_01x01_Pin") (at 328.295 243.205 0) (unit 1)
-    (in_bom yes) (on_board yes) (dnp no) (fields_autoplaced)
+    (in_bom no) (on_board yes) (dnp no) (fields_autoplaced)
     (property "Reference" "J6" (at 328.93 239.395 0)
       (effects (font (size 1.27 1.27)))
@@
   )
   (symbol (lib_id "Lora:pcb_antenna") (at 235.585 142.24 0) (unit 1)
-    (in_bom yes) (on_board yes) (dnp no) (fields_autoplaced)
+    (in_bom no) (on_board yes) (dnp no) (fields_autoplaced)
     (property "Reference" "PCB_Antenna1" (at 243.205 142.875 0)
       (effects (font (size 1.27 1.27)) (justify left))
@@
   )
   (symbol (lib_id "Connector:Conn_01x08_Pin") (at 320.04 55.88 0) (unit 1)
-    (in_bom yes) (on_board yes) (dnp no)
+    (in_bom no) (on_board yes) (dnp no)
     (property "Reference" "J5" (at 322.58 44.45 0)
       (effects (font (size 1.27 1.27)))
