File: hardware/winch-link/winch-link.kicad_pcb (KiCad board)
At the start: 2 copper layers, 80 x 45 mm, 45 parts, among them J1 USB_C_Receptacle_USB2.0, J2 Conn_01x02_Pin, J3 Conn_01x02_Pin, J4 VBAT, J5 display conn, J6 BAT GND, Q1 AO3401A, SW1 RST, SW2 PRG, U1 RFM95W-868S2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

Commit message: Add BOM and CPL files
Changed lines of the file:
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@@
       (plot_on_all_layers_selection 0x0000000_00000000)
       (disableapertmacros false)
-      (usegerberextensions false)
-      (usegerberattributes true)
-      (usegerberadvancedattributes true)
-      (creategerberjobfile true)
+      (usegerberextensions true)
+      (usegerberattributes false)
+      (usegerberadvancedattributes false)
+      (creategerberjobfile false)
       (dashed_line_dash_ratio 12.000000)
       (dashed_line_gap_ratio 3.000000)
@@
       (psa4output false)
       (plotreference true)
-      (plotvalue true)
+      (plotvalue false)
       (plotinvisibletext false)
       (sketchpadsonfab false)
-      (subtractmaskfromsilk false)
+      (subtractmaskfromsilk true)
       (outputformat 1)
       (mirror false)
-      (drillshape 1)
+      (drillshape 0)
       (scaleselection 1)
-      (outputdirectory "")
+      (outputdirectory "Gerber/")
     )
   )
@@
     (effects (font (size 5 5) (thickness 1) bold))
   )
-  (gr_text "winch link" (at 169.37868 109.87868 270) (layer "F.SilkS")
+  (gr_text "winch link" (at 169.37868 110.75 270) (layer "F.SilkS")
     (effects (font (size 4 4) (thickness 0.6) bold))
   )

Commit message: Add README.md
Other:
- board text added: "github.com/martinpetri/winch-link"
- board text added: "version 1.0"
